File: boardswap.kicad_pcb (KiCad board)
At the start: 2 copper layers, 285 x 96.1 mm, 155 parts, among them J1 USB_C_Receptacle_USB2.0, SW1 SW_Push, U1 ATmega32U4-AU, Y1 16MHz

Commit message: did most placement
Parts:
- C7: footprint Diode_SMD:D_SOD-123 -> Capacitor_SMD:C_0805_2012Metric
- D29, D30, D31, D32, D33, D34, D35, D36, D37, D38, D39, D40, D41, D42, D43, D44, D45, D46, D47, D48, D49, D50, D51, D52, D53, D54, D55, D56, D57, D58, D59, D60, D61, D62, D63, D64, D65, D66, D67, D68, F1, J1, SW1, U1: moved to B.Cu
- moved REF** 444.5 mm to (123.8, -176.2)
- moved D56 315.9 mm to (246.1, -152.4), turned to 90 degrees
- moved D42 307.6 mm to (246.1, -171.4), turned to 90 degrees
- moved D67 297.9 mm to (222.2, -133.3), turned to 90 degrees
- moved D68 287.0 mm to (246.1, -133.3), turned to 90 degrees
- moved D41 278.0 mm to (222.2, -171.4), turned to 90 degrees
- moved D39 268.6 mm to (184.2, -171.4), turned to 90 degrees
- moved D55 263.2 mm to (222.2, -152.4), turned to 90 degrees
- moved D40 258.9 mm to (203.2, -171.4), turned to 90 degrees
- moved D65 249.9 mm to (184.2, -133.3), turned to 90 degrees
- moved D66 246.0 mm to (203.2, -133.3), turned to 90 degrees
- moved D54 238.6 mm to (203.2, -152.4), turned to 90 degrees
- moved D64 236.3 mm to (165.1, -133.3), turned to 90 degrees
- moved D51 225.5 mm to (146.1, -152.4), turned to 90 degrees
- moved D52 223.5 mm to (165.1, -152.4), turned to 90 degrees
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Other:
- net class Default: trace_width 0.25 -> 0.254
- net class Power added: clearance 0.2, trace_width 0.381, via_dia 0.8, via_drill 0.4
