File: boardswap.kicad_pcb (KiCad board)
At the start: 2 copper layers, 285 x 96.1 mm, 157 parts, among them J1 USB_C_Receptacle_USB2.0, SW1 SW_Push, U1 ATmega32U4-AU, Y1 16MHz

Commit message: added more stuff
Parts:
- MX1, MX10, MX11, MX12, MX13, MX14, MX15, MX16, MX17, MX18, MX19, MX2, MX20, MX21, MX22, MX23, MX24, MX25, MX26, MX27, MX28, MX29, MX3, MX30, MX31, MX32, MX33, MX34, MX35, MX36, MX37, MX38, MX39, MX4, MX40, MX41, MX42, MX43, MX44, MX45, MX46, MX47, MX48, MX49, MX5, MX50, MX51, MX52, MX53, MX54, MX55, MX56, MX57, MX58, MX59, MX6, MX60, MX61, MX62, MX63, MX64, MX65, MX66, MX67, MX68, MX7, MX8, MX9: footprint keyswitches:Kailh_socket_MX_alt -> switchprint:Kailh_socket_MX_alt
- moved C1 266.2 mm to (40.2, 119.0)
- moved C2 266.2 mm to (43.9, 116.5)
- moved C3 266.2 mm to (26.6, 104.8)
- moved C4 266.2 mm to (29.2, 105.5)
- moved C5 266.2 mm to (29.2, 104.0)
- moved C6 266.2 mm to (19.5, 118.4)
- moved C7 266.2 mm to (21.2, 118.5)
- moved D1 266.2 mm to (10.6, 46.2)
- moved D10 266.2 mm to (193.2, 55.8)
- moved D11 266.2 mm to (212.3, 55.8)
- moved D12 266.2 mm to (231.3, 55.8)
- moved D13 266.2 mm to (250.4, 55.8)
- moved D14 266.2 mm to (274.2, 55.8)
- moved D15 266.2 mm to (17.0, 74.8)
- moved D16 266.2 mm to (40.8, 74.8)
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
Commit message: made everything nice
Parts:
- removed the REF** at (145.6, 89.1)
- added G***: LOGO, logo:logo, F.Cu at (146.7, 90.1)
- added OUTLINE: 60_Outline, locallib:60_Outline-Modded, F.Cu at (145.6, 89.1)
- moved R2 1.89 mm to (28.8, 54.9)
- moved R3 0.23 mm to (26.7, 57.1)
Routing:
- net Net-(R2-Pad1): track 56.4 -> 67.9 mm
- net D+: track 15.7 -> 13.8 mm

Commit message: prettified logo
Parts:
- moved G*** 3.25 mm to (145.8, 86.9)

Commit message: pretty logo
Parts:
- moved G*** 21.6 mm to (164.4, 75.9)
